Commit message: new description

File: robot_description/urdf/pan_tilt.urdf (robot description, URDF)
Before this commit: robot pan_tilt, 3 links, 2 joints
Links:
- link base_link: geometry collision cylinder length=0.2 radius=0.3; visual cylinder length=0.1 radius=0.02
Joints:
- joint tilt_joint: limit lower=-4.64 upper=-1.5 effort=300.0 velocity=0.1 -> lower=-4.64 upper=3.14 effort=300.0 velocity=0.1; origin xyz=0.0 0.0 0.2 -> xyz=0.0 0.0 0.4
