Commit message: updated

File: robot_description/urdf/seven_dof_arm.xacro (robot description, xacro)
@@ -51,5 +51,6 @@
     <xacro:property name="elbow_pitch_height" value="0.04" />
     <!-- Wrist roll link properties -->
-    <xacro:property name="wrist_roll_width" value="0.02" />
+    <xacro:property name="wrist_roll_width" value="bottom_link
+No transform from [bottom_link] to [base_link]0.02" />
     <xacro:property name="wrist_roll_len" value="0.04" />
     <!-- wrist pitch link properties -->
@@ -195,5 +196,6 @@
     <gazebo reference="shoulder_pitch_link">
         <material>Gazebo/White</material>
-    </gazebo>
+    </gazebo>from distutils.core import setup
+from setuptools import find_packages
     <joint name="elbow_roll_joint" type="revolute">
         <parent link="shoulder_pitch_link"/>
@@ -415,3 +417,20 @@
     </joint>
     <xacro:include filename="$(find robot_description)/urdf/sensors/xtion_pro_live.urdf.xacro"/>
+    <!-- ///////////////////////////////////////////////////////////////////////////////////////////////////////////////////// -->
+    <!-- Transmissions for ROS Control -->
+    <xacro:transmission_block joint_name="shoulder_pan_joint"/>
+    <xacro:transmission_block joint_name="shoulder_pitch_joint"/>
+    <xacro:transmission_block joint_name="elbow_roll_joint"/>
+    <xacro:transmission_block joint_name="elbow_pitch_joint"/>
+    <xacro:transmission_block joint_name="wrist_roll_joint"/>
+    <xacro:transmission_block joint_name="wrist_pitch_joint"/>
+    <xacro:transmission_block joint_name="gripper_roll_joint"/>
+    <xacro:transmission_block joint_name="finger_joint1"/>
+    <xacro:transmission_block joint_name="finger_joint2"/>
+    <!-- ros_control plugin -->
+    <gazebo>
+        <plugin name="gazebo_ros_control" filename="libgazebo_ros_control.so">
+        <robotNamespace>/seven_dof_arm</robotNamespace>
+        </plugin>
+    </gazebo>
 </robot>
