Commit message: twicks here and there

File: a05_seven_dof_arm/urdf/seven_dof_arm_with_rgbd.xacro (robot description, xacro)
@@ -1,163 +1,23 @@
-<?xml version="1.0"?>
-<robot xmlns:xacro="http://www.ros.org/wiki/xacro" name="seven_dof_arm">
-    <!-- rgbd sensor file -->
-	<xacro:include filename="$(find a05_seven_dof_arm)/urdf/sensors/xtion_pro_live.urdf.xacro"/>
-    <!-- Include materials -->
-    <material name="Black">
-        <color rgba="0.0 0.0 0.0 1.0"/>
-    </material>
-    <material name="Red">
-        <color rgba="0.8 0.0 0.0 1.0"/>
-    </material>
-    <material name="White">
-        <color rgba="1.0 1.0 1.0 1.0"/>
-    </material>
-    <material name="Blue">
-        <color rgba="0.0 0.0 0.8 1.0"/>
-    </material>
-    <material name="Green">
-        <color rgba="0.0 0.8 0.0 1.0"/>
-    </material>
-    <material name="Yellow">
-        <color rgba="1.0 1.0 0.0 1.0"/>
-    </material>
-    <material name="Cyan">
-        <color rgba="0.0 1.0 1.0 1.0"/>
-    </material>
-    <material name="Magenta">
-        <color rgba="1.0 0.0 1.0 1.0"/>
-    </material>
-    <material name="Gray">
-        <color rgba="0.5 0.5 0.5 1.0"/>
-    </material>
-    <material name="Orange">
-        <color rgba="1.0 0.5 0.0 1.0"/>
-    </material>
-    <!-- Constants -->
-    <xacro:property name="M_PI" value="3.14159"/>
-    <xacro:property name="M_SCALE" value="0.001 0.001 0.001"/>
-    <xacro:property name="deg_to_rad" value="0.01745329251994329577"/>
-    <!-- Shoulder pan link properties -->
-    <xacro:property name="shoulder_pan_width" value="0.04" />
-    <xacro:property name="shoulder_pan_len" value="0.08" />
-    <!-- Shoulder pitch link properties -->
-    <xacro:property name="shoulder_pitch_len" value="0.14" />
-    <xacro:property name="shoulder_pitch_width" value="0.04" />
-    <xacro:property name="shoulder_pitch_height" value="0.04" />
-    <!-- Elbow roll link properties -->
-    <xacro:property name="elbow_roll_width" value="0.02" />
-    <xacro:property name="elbow_roll_len" value="0.06" />
-    <!-- Elbow pitch link properties -->
-    <xacro:property name="elbow_pitch_len" value="0.22" />
-    <xacro:property name="elbow_pitch_width" value="0.04" />
-    <xacro:property name="elbow_pitch_height" value="0.04" />
-    <!-- Wrist roll link properties -->
-    <xacro:property name="wrist_roll_width" value="0.02" />
-    <xacro:property name="wrist_roll_len" value="0.04" />
-    <!-- wrist pitch link properties -->
-    <xacro:property name="wrist_pitch_len" value="0.06" />
-    <xacro:property name="wrist_pitch_width" value="0.04" />
-    <xacro:property name="wrist_pitch_height" value="0.04" />
-    <!-- Gripper roll link properties -->
-    <xacro:property name="gripper_roll_width" value="0.04" />
-    <xacro:property name="gripper_roll_len" value="0.02" />
-    <!-- Left gripper -->
-    <xacro:property name="left_gripper_len" value="0.08" />
-    <xacro:property name="left_gripper_width" value="0.01" />
-    <xacro:property name="left_gripper_height" value="0.01" />
-    <!-- Right gripper -->
-    <xacro:property name="right_gripper_len" value="0.08" />
-    <xacro:property name="right_gripper_width" value="0.01" />
-    <xacro:property name="right_gripper_height" value="0.01" />
-    <!-- macros: kind of like struct in c -->
-    <xacro:macro name="inertial_matrix" params="mass">
-        <inertial>
-            <mass value="${mass}"/>
-            <inertia ixx="0.5" ixy="0.0" ixz="0.0" iyy="0.5" iyz="0.0" izz="0.5"/>
-        </inertial>
-    </xacro:macro>
-    <xacro:macro name="transmission_block" params="joint_name">
-        <transmission name="${joint_name}_trans">
-            <type>transmission_interface/SimpleTransmission</type>
-            <joint name="${joint_name}">
-                <hardwareInterface>hardware_interface/PositionJointInterface</hardwareInterface>
-            </joint>
-            <actuator name="${joint_name}_motor">
-                <mechanicalReduction>1.0</mechanicalReduction>
-                <hardwareInterface>hardware_interface/PositionJointInterface</hardwareInterface>
-            </actuator>
-        </transmission>
-    </xacro:macro>
-    <!-- /////////////////////////////////////////////////////////////////////// -->
-    <!-- base_link -->
-    <link name="base_link">
-        <visual>
-            <origin xyz="0.0 0.0 0.0" rpy="${M_PI/2} 0.0 0.0"/>
-            <geometry>
-                <box size="0.10 0.10 0.10"/>
-            </geometry>
-            <material name="White">
-            </material>
-        </visual>
-        <collision>
-            <origin xyz="0.0 0.0 0.0" rpy="${M_PI/2} 0.0 0.0"/>
-            <geometry>
-                <box size="0.10 0.10 0.10"/>
-            </geometry>
-        </collision>
-        <!-- <xacro:inertial_matrix mass="1"/> -->
-    </link>
-    <gazebo reference = "base_link">
-        <material>Gazebo/White</material>
-    </gazebo>
-    <!-- /////////////////////////////////////////////////////////////////////// -->
-    <!-- bottom_joint -->
-    <joint name="bottom_joint" type="fixed">
-        <origin xyz="0.0 0.0 0.0" rpy="0.0 0.0 0.0"/>
-        <parent link="base_link"/>
-        <child link="bottom_link"/>
-    </joint>
-    <!-- bottom_link -->
-    <link name="bottom_link">
-        <visual>
-            <origin xyz="0.0 0.0 -0.04" rpy="0.0 0.0 0.0"/>
-            <geometry>
-                <box size="1 1 0.02"/>
-            </geometry>
-            <material name="Yellow">
-            </material>
-        </visual>
-        <collision>
-            <origin xyz="0.0 0.0 -0.04" rpy="0.0 0.0 0.0"/>
-            <geometry>
-                <box size="1 1 0.02"/>
-            </geometry>
-        </collision>
-    </link>
-    <gazebo reference="bottom_link">
-        <material>Gazebo/Yellow</material>
-    </gazebo>
-    <!-- /////////////////////////////////////////////////////////////////////// -->
-    <!-- sholder_pan_joint -->
-    <joint name="shoulder_pan_joint" type="revolute">
-        <origin xyz="0.0 0.0 0.05" rpy="0.0 ${M_PI/2} 0"/>
+<!-- ///////////////////////////////////////////////////////////////////////////////////////////////////////////////////// -->
+    <joint name="shoulder_pan_joint1" type="revolute">
         <parent link="base_link"/>
         <child link="shoulder_pan_link"/>
-        <axis xyz="-1 0.0 0"/>
-        <limit lower="-2.61" upper="1.98" effort="300.0" velocity="1.0"/>
-        <!-- <dynamics damping="50" friction="1"/> -->
-    </joint>
-    <!-- shoulder_pan_link -->
-    <link name="shoulder_pan_link">
-        <visual>
-            <origin xyz="0.0 0.0 0" rpy="0.0 ${M_PI/2} 0.0"/>
+        <origin xyz="0 0 0.05" rpy="0 ${M_PI/2} ${M_PI*0}" />
+        <axis xyz="-1 0 0" />
+        <limit effort="300" velocity="1" lower="-2.61799387799" upper="1.98394848567"/>
+        <dynamics damping="50" friction="1"/>
+    </joint>
+<!-- ///////////////////////////////////////////////////////////////////////////////////////////////////////////////////// -->
+  <!-- SHOULDER PAN LINK -->
+    <link name="shoulder_pan_link" >
+        <visual>
+            <origin xyz="0 0 0" rpy="0 ${M_PI/2} 0" />
             <geometry>
                 <cylinder radius="${shoulder_pan_width}" length="${shoulder_pan_len}"/>
             </geometry>
-            <material name="Red">
-            </material>
-        </visual>
-        <collision>
-            <origin xyz="0.0 0.0 0.0" rpy="0.0 ${M_PI/2} 0.0"/>
+            <material name="Red" />
+        </visual>
+        <collision>
+            <origin xyz="0 0 0" rpy="0 ${M_PI/2} 0" />
             <geometry>
                 <cylinder radius="${shoulder_pan_width}" length="${shoulder_pan_len}"/>
@@ -177,19 +37,19 @@
         <dynamics damping="50" friction="1"/>
     </joint>
-    <!-- ///////////////////////////////////////////////////////////////////////////////////////////////////////////////////// -->
-    <!-- SHOULDER PITCH LINK -->
+<!-- ///////////////////////////////////////////////////////////////////////////////////////////////////////////////////// -->
+  <!-- SHOULDER PITCH LINK -->
     <link name="shoulder_pitch_link" >
         <visual>
-        <origin xyz="-0.002 0 0.04" rpy="0 ${M_PI/2} 0" />
-        <geometry>
-            <box size="${shoulder_pitch_len} ${shoulder_pitch_width} ${shoulder_pitch_height}" />
-        </geometry>
-        <material name="White" />
-        </visual>
-        <collision>
-        <origin xyz="-0.002 0 0.04" rpy="0 ${M_PI/2} 0" />
-        <geometry>
-            <box size="${shoulder_pitch_len} ${shoulder_pitch_width} ${shoulder_pitch_height}" />
-        </geometry>
+            <origin xyz="-0.002 0 0.04" rpy="0 ${M_PI/2} 0" />
+            <geometry>
+                <box size="${shoulder_pitch_len} ${shoulder_pitch_width} ${shoulder_pitch_height}" />
+            </geometry>
+            <material name="White" />
+        </visual>
+        <collision>
+            <origin xyz="-0.002 0 0.04" rpy="0 ${M_PI/2} 0" />
+            <geometry>
+                <box size="${shoulder_pitch_len} ${shoulder_pitch_width} ${shoulder_pitch_height}" />
+            </geometry>
         </collision>
         <xacro:inertial_matrix mass="1"/>
@@ -206,19 +66,19 @@
         <dynamics damping="50" friction="1"/>
     </joint>
-    <!-- ///////////////////////////////////////////////////////////////////////////////////////////////////////////////////// -->
+<!-- ///////////////////////////////////////////////////////////////////////////////////////////////////////////////////// -->
     <!-- ELBOW ROLL LINK -->
     <link name="elbow_roll_link" >
         <visual>
-        <origin xyz="-0.015 0.0 -0.0" rpy="0 ${M_PI/2} 0" />
-        <geometry>
-                <cylinder radius="${elbow_roll_width}" length="${elbow_roll_len}"/>
-        </geometry>
-        <material name="Black" />
-        </visual>
-        <collision>
-        <origin xyz="-0.015 0.0 -0.0" rpy="0 ${M_PI/2} 0" />
-        <geometry>
-                <cylinder radius="${elbow_roll_width}" length="${elbow_roll_len}"/>
-        </geometry>
+            <origin xyz="-0.015 0.0 -0.0" rpy="0 ${M_PI/2} 0" />
+            <geometry>
+                <cylinder radius="${elbow_roll_width}" length="${elbow_roll_len}"/>
+            </geometry>
+            <material name="Black" />
+        </visual>
+        <collision>
+            <origin xyz="-0.015 0.0 -0.0" rpy="0 ${M_PI/2} 0" />
+            <geometry>
+                <cylinder radius="${elbow_roll_width}" length="${elbow_roll_len}"/>
+            </geometry>
         </collision>
         <xacro:inertial_matrix mass="1"/>
@@ -235,19 +95,19 @@
         <dynamics damping="50" friction="1"/>
     </joint>
-    <!-- ///////////////////////////////////////////////////////////////////////////////////////////////////////////////////// -->
+<!-- ///////////////////////////////////////////////////////////////////////////////////////////////////////////////////// -->
     <!-- ELBOW PITCH LINK -->
     <link name="elbow_pitch_link" >
         <visual>
-        <origin xyz="0 0 -0.12" rpy="0 ${M_PI/2} 0" />
-        <geometry>
-        <box size="${elbow_pitch_len} ${elbow_pitch_width} ${elbow_pitch_height}" />
-        </geometry>
-        <material name="Red" />
-        </visual>
-        <collision>
-        <origin xyz="0 0 -0.12" rpy="0 ${M_PI/2} 0" />
-        <geometry>
-        <box size="${elbow_pitch_len} ${elbow_pitch_width} ${elbow_pitch_height}" />
-        </geometry>
+            <origin xyz="0 0 -0.12" rpy="0 ${M_PI/2} 0" />
+            <geometry>
+            <box size="${elbow_pitch_len} ${elbow_pitch_width} ${elbow_pitch_height}" />
+            </geometry>
+            <material name="Red" />
+        </visual>
+        <collision>
+            <origin xyz="0 0 -0.12" rpy="0 ${M_PI/2} 0" />
+            <geometry>
+            <box size="${elbow_pitch_len} ${elbow_pitch_width} ${elbow_pitch_height}" />
+            </geometry>
         </collision>
         <xacro:inertial_matrix mass="1"/>
@@ -264,18 +124,19 @@
         <dynamics damping="50" friction="1"/>
     </joint>
+<!-- ///////////////////////////////////////////////////////////////////////////////////////////////////////////////////// -->
     <!-- WRIST ROLL LINK -->
     <link name="wrist_roll_link" >
         <visual>
-        <origin xyz="0 0 0" rpy="0 ${M_PI/2} 0" />
-        <geometry>
-            <cylinder radius="${elbow_roll_width}" length="${elbow_roll_len}"/>
-        </geometry>
-        <material name="Black" />
-        </visual>
-        <collision>
-        <origin xyz="0 0 0" rpy="0 ${M_PI/2} 0" />
-        <geometry>
-            <cylinder radius="${elbow_roll_width}" length="${elbow_roll_len}"/>
-        </geometry>
+            <origin xyz="0 0 0" rpy="0 ${M_PI/2} 0" />
+            <geometry>
+                <cylinder radius="${elbow_roll_width}" length="${elbow_roll_len}"/>
+            </geometry>
+            <material name="Black" />
+        </visual>
+        <collision>
+            <origin xyz="0 0 0" rpy="0 ${M_PI/2} 0" />
+            <geometry>
+                <cylinder radius="${elbow_roll_width}" length="${elbow_roll_len}"/>
+            </geometry>
         </collision>
         <xacro:inertial_matrix mass="1"/>
@@ -284,5 +145,5 @@
         <material>Gazebo/Black</material>
     </gazebo>
-     <joint name="wrist_pitch_joint" type="revolute">
+    <joint name="wrist_pitch_joint" type="revolute">
         <parent link="wrist_roll_link"/>
         <child link="wrist_pitch_link"/>
@@ -292,19 +153,19 @@
         <dynamics damping="50" friction="1"/>
     </joint>
-    <!-- ///////////////////////////////////////////////////////////////////////////////////////////////////////////////////// -->
+<!-- ///////////////////////////////////////////////////////////////////////////////////////////////////////////////////// -->
     <!-- WRIST PITCH LINK -->
     <link name="wrist_pitch_link">
         <visual>
-        <origin xyz="0 0 0.04" rpy="0 ${M_PI/2} 0" />
-        <geometry>
-            <box size="${wrist_pitch_len} ${wrist_pitch_width} ${wrist_pitch_height}" />
-        </geometry>
-        <material name="White" />
-        </visual>
-        <collision>
-        <origin xyz="0 0 0.04 " rpy="0 ${M_PI/2} 0" />
-        <geometry>
-            <box size="${wrist_pitch_len} ${wrist_pitch_width} ${wrist_pitch_height}" />
-        </geometry>
+            <origin xyz="0 0 0.04" rpy="0 ${M_PI/2} 0" />
+            <geometry>
+                <box size="${wrist_pitch_len} ${wrist_pitch_width} ${wrist_pitch_height}" />
+            </geometry>
+            <material name="White" />
+        </visual>
+        <collision>
+            <origin xyz="0 0 0.04 " rpy="0 ${M_PI/2} 0" />
+            <geometry>
+                <box size="${wrist_pitch_len} ${wrist_pitch_width} ${wrist_pitch_height}" />
+            </geometry>
         </collision>
         <xacro:inertial_matrix mass="1"/>
@@ -318,25 +179,22 @@
         <origin xyz="0 0 0.080" rpy="${1.5*M_PI} -${.5*M_PI} 0" />
         <axis xyz="1 0 0" />
-        <!--
-            <limit effort="300" velocity="1" lower="-2.61799387799" upper="2.6128806087" />
-            -->
-            <limit effort="300" velocity="1" lower="-3.14" upper="3.14" />
-        <dynamics damping="50" friction="1"/>
-    </joint>
-    <!-- ///////////////////////////////////////////////////////////////////////////////////////////////////////////////////// -->
+        <limit effort="300" velocity="1" lower="-2.61799387799" upper="2.6128806087" />
+        <dynamics damping="50" friction="1"/>
+    </joint>
+<!-- ///////////////////////////////////////////////////////////////////////////////////////////////////////////////////// -->
     <!-- GRIPPER ROLL LINK -->
     <link name="gripper_roll_link">
         <visual>
-        <origin xyz="0 0 0" rpy="0 ${M_PI/2} 0" />
-        <geometry>
+            <origin xyz="0 0 0" rpy="0 ${M_PI/2} 0" />
+            <geometry>
                 <cylinder radius="${gripper_roll_width}" length="${gripper_roll_len}"/>
-        </geometry>
-        <material name="Red" />
-        </visual>
-        <collision>
-        <origin xyz="0 0 0" rpy="0 ${M_PI/2} 0" />
-        <geometry>
+            </geometry>
+            <material name="Red" />
+        </visual>
+        <collision>
+            <origin xyz="0 0 0" rpy="0 ${M_PI/2} 0" />
+            <geometry>
                 <cylinder radius="${gripper_roll_width}" length="${gripper_roll_len}"/>
-        </geometry>
+            </geometry>
         </collision>
         <xacro:inertial_matrix mass="1"/>
@@ -350,16 +208,20 @@
         <origin xyz="0.0 0 0" />
         <axis xyz="0 1 0" />
-        <limit effort="1" lower="0" upper="0.03" velocity="1.0"/>
-        <dynamics damping="50" friction="1"/>
-    </joint>
-    <!-- ///////////////////////////////////////////////////////////////////////////////////////////////////////////////////// -->
+            <limit effort="100" lower="0" upper="0.03" velocity="1.0"/>
+            <safety_controller k_position="20"
+                                k_velocity="20"
+                                soft_lower_limit="${-0.15 }"
+                                soft_upper_limit="${ 0.0 }"/>
+        <dynamics damping="50" friction="1"/>
+    </joint>
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