Commit message: ros control in gazebo

File: a05_seven_dof_arm/urdf/sensors/xtion_pro_live.gazebo.xacro (robot description, xacro)
@@ -3,6 +3,6 @@
   <xacro:macro name="xtion_pro_live_rgbd_camera_gazebo" params="name">
     <gazebo reference="${name}_link">
-      <!-- Depth (IR) -->
-      <sensor type="depth" name="${name}_frame_sensor">
+      <!-- Depth (IR) Sensor -->
+      <sensor type="depth" name="${name}_depth_frame_sensor">
         <always_on>true</always_on>
         <update_rate>6.0</update_rate>
@@ -19,5 +19,5 @@
           </clip>
         </camera>
-        <plugin name="${name}_frame_controller" filename="libgazebo_ros_openni_kinect.so">
+        <plugin name="${name}_depth_frame_controller" filename="libgazebo_ros_openni_kinect.so">
           <alwaysOn>true</alwaysOn>
           <updateRate>6.0</updateRate>
@@ -33,13 +33,15 @@
           <rangeMax>1.5</rangeMax>
           <!-- Distortion parameters not supported in gazebo 1.9.* plugins -->
-          <!--distortionK1>0.00000001</distortionK1>
+          <!--
+          <distortionK1>0.00000001</distortionK1>
           <distortionK2>0.00000001</distortionK2>
           <distortionK3>0.00000001</distortionK3>
           <distortionT1>0.00000001</distortionT1>
-          <distortionT2>0.00000001</distortionT2-->
+          <distortionT2>0.00000001</distortionT2>
+          -->
         </plugin>
       </sensor>
-      <!-- RGB -->
-      <sensor type="depth" name="${name}_frame_sensor">
+      <!-- RGB Sensor -->
+      <sensor type="camera" name="${name}_rgb_frame_sensor">
         <always_on>true</always_on>
         <update_rate>6.0</update_rate>
@@ -56,5 +58,5 @@
           </clip>
         </camera>
-        <plugin name="${name}_frame_controller" filename="libgazebo_ros_openni_kinect.so">
+        <plugin name="${name}_rgb_frame_controller" filename="libgazebo_ros_camera.so">
           <alwaysOn>true</alwaysOn>
           <updateRate>6.0</updateRate>
@@ -62,13 +64,7 @@
           <imageTopicName>rgb/image_raw</imageTopicName>
           <cameraInfoTopicName>rgb/camera_info</cameraInfoTopicName>
-          <pointCloudTopicName>rgb/points</pointCloudTopicName>
-          <depthImageTopicName>depth/image_raw</depthImageTopicName>
-          <depthImageCameraInfoTopicName>depth/camera_info</depthImageCameraInfoTopicName>
           <frameName>${name}_optical_frame</frameName>
-          <pointCloudCutoff>0.05</pointCloudCutoff>
-          <pointCloudCutoffMax>5</pointCloudCutoffMax>
-          <rangeMax>1.5</rangeMax>
         </plugin>
-     </sensor>
+      </sensor>
     </gazebo>
   </xacro:macro>

File: a05_seven_dof_arm/urdf/sensors/xtion_pro_live.urdf.xacro (robot description, xacro)
@@ -1,5 +1,7 @@
 <?xml version="1.0"?>
 <robot xmlns:xacro="http://ros.org/wiki/xacro">
+  <!-- Include Gazebo-specific elements -->
   <xacro:include filename="$(find a05_seven_dof_arm)/urdf/sensors/xtion_pro_live.gazebo.xacro"/>
+  <!-- Define a macro for dummy inertial properties -->
   <xacro:macro name="dummy_inertial">
     <inertial>
@@ -11,6 +13,7 @@
     </inertial>
   </xacro:macro>
+  <!-- Main macro definition for xtion_pro_live sensor -->
   <xacro:macro name="xtion_pro_live" params="name parent *origin *optical_origin">
-    <!-- frames in the center of the camera -->
+    <!-- Main sensor link -->
     <joint name="${name}_joint" type="fixed">
       <xacro:insert_block name="origin"/>
@@ -27,21 +30,20 @@
       </inertial>
       <visual>
-         <geometry>
-          <!--
-          <box size="0.06 0.1 0.03" />
-        	-->
-					<mesh filename="package://a05_seven_dof_arm/meshes/sensors/xtion_pro_live/xtion_pro_live.stl"/>
+        <geometry>
+          <mesh filename="package://a05_seven_dof_arm/meshes/sensors/xtion_pro_live/xtion_pro_live.stl"/>
         </geometry>
-        <material name="Blue"/>
+        <material name="White"/>
       </visual>
       <collision>
-      <geometry>
+        <geometry>
           <mesh filename="package://a05_seven_dof_arm/meshes/sensors/xtion_pro_live/xtion_pro_live.dae"/>
-      </geometry>
+        </geometry>
       </collision>
     </link>
+    <!-- Gazebo-specific color -->
     <gazebo reference="${name}_link">
-      <material>Gazebo/Blue</material>
+      <material>Gazebo/White</material>
     </gazebo>
+    <!-- Optical frame -->
     <joint name="${name}_optical_joint" type="fixed">
       <xacro:insert_block name="optical_origin"/>
@@ -50,5 +52,5 @@
     </joint>
     <link name="${name}_optical_frame">
-      <dummy_inertial/>
+      <xacro:dummy_inertial/>
     </link>
     <!-- Depth sensor frames -->
@@ -59,5 +61,5 @@
     </joint>
     <link name="${name}_depth_frame">
-      <dummy_inertial/>
+      <xacro:dummy_inertial/>
     </link>
     <joint name="${name}_depth_optical_joint" type="fixed">
@@ -67,5 +69,5 @@
     </joint>
     <link name="${name}_depth_optical_frame">
-      <dummy_inertial/>
+      <xacro:dummy_inertial/>
     </link>
     <!-- RGB sensor frames -->
@@ -76,5 +78,5 @@
     </joint>
     <link name="${name}_rgb_frame">
-      <dummy_inertial/>
+      <xacro:dummy_inertial/>
     </link>
     <joint name="${name}_rgb_optical_joint" type="fixed">
@@ -84,7 +86,7 @@
     </joint>
     <link name="${name}_rgb_optical_frame">
-      <dummy_inertial/>
+      <xacro:dummy_inertial/>
     </link>
-    <!-- <xacro:xtion_pro_live_rgbd_camera_gazebo name="${name}"/> -->
+    <xacro:xtion_pro_live_rgbd_camera_gazebo name="${name}"/>
   </xacro:macro>
 </robot>

File: a05_seven_dof_arm/urdf/seven_dof_arm.xacro (robot description, xacro)
@@ -2,5 +2,5 @@
 <robot name="seven_dof_arm" xmlns:xacro="http://ros.org/wiki/xacro">
     <!-- rgbd sensor file -->
-    <!-- <xacro:include filename="$(find a05_seven_dof_arm)/urdf/sensors/xtion_pro_live.urdf.xacro"/> -->
+    <xacro:include filename="$(find a05_seven_dof_arm)/urdf/sensors/xtion_pro_live.urdf.xacro"/>
 	<!-- Include materials -->
     <material name="Black">
@@ -87,5 +87,6 @@
             </geometry>
         </collision>
-    <!-- <xacro:inertial_matrix mass="1"/> -->
+<!-- you idiot always put inertia inertia inertia -->
+        <xacro:inertial_matrix mass="1"/>
     </link>
     <gazebo reference="base_link">
@@ -120,5 +121,5 @@
     </gazebo>
 <!-- ///////////////////////////////////////////////////////////////////////////////////////////////////////////////////// -->
-    <joint name="shoulder_pan_joint1" type="revolute">
+    <joint name="shoulder_pan_joint" type="revolute">
         <parent link="base_link"/>
         <child link="shoulder_pan_link"/>
@@ -376,10 +377,10 @@
 <!-- ///////////////////////////////////////////////////////////////////////////////////////////////////////////////////// -->
     <!-- Define RGB-D sensor -->
-    <!-- <xacro:xtion_pro_live name="rgbd_camera" parent="base">
+    <xacro:xtion_pro_live name="rgbd_camera" parent="base">
         <origin xyz="0.1 0.0 0.9" rpy="${0.0 * deg_to_rad} ${70.0 * deg_to_rad} ${0.0 * deg_to_rad}"/>
-        <origin xyz="0 0 0" rpy="${-90 * deg_to_rad} ${0 * deg_to_rad} ${-90 * deg_to_rad}" />
-    </xacro:xtion_pro_live> -->
+        <optical_origin xyz="0 0 0" rpy="${-90 * deg_to_rad} ${0 * deg_to_rad} ${-90 * deg_to_rad}" />
+    </xacro:xtion_pro_live>
     <!-- Transmissions for ROS Control -->
-    <!-- <xacro:transmission_block joint_name="shoulder_pan_joint"/>
+    <xacro:transmission_block joint_name="shoulder_pan_joint"/>
     <xacro:transmission_block joint_name="shoulder_pitch_joint"/>
     <xacro:transmission_block joint_name="elbow_roll_joint"/>
@@ -389,10 +390,10 @@
     <xacro:transmission_block joint_name="gripper_roll_joint"/>
     <xacro:transmission_block joint_name="finger_joint1"/>
-    <xacro:transmission_block joint_name="finger_joint2"/> -->
+    <xacro:transmission_block joint_name="finger_joint2"/>
     <!-- ros_control plugin -->
-    <!-- <gazebo>
+    <gazebo>
         <plugin name="gazebo_ros_control" filename="libgazebo_ros_control.so">
             <robotNamespace>/seven_dof_arm</robotNamespace>
         </plugin>
-    </gazebo> -->
+    </gazebo>
 </robot>
